File: Pi_HIL/Pi_HIL.kicad_pcb (KiCad board)
At the start: 2 copper layers, 65 x 56.5 mm, 45 parts, among them J1 Raspberry_Pi_2_3, J2 Conn_01x04_Male, J3 Conn_01x04_Male, J4 Conn_01x02_Male, J5 Conn_01x02_Male, J6 Conn_01x03, Q1 MMBT3904, U1 B0505LS-1WR3, U2 ADuM1250ARZ, U3 AMS1117-3.3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

Commit message: Updated Layout + Schematic
Parts:
- C2: moved to F.Cu
- moved U4 92.5 mm to (134.0, 85.8)
- moved J3 73.3 mm to (161.8, 75.8)
- moved J2 66.5 mm to (153.5, 79.5)
- moved J4 60.3 mm to (157.7, 84.5)
- moved C6 56.5 mm to (138.5, 86.0), turned to -90 degrees
- moved JP1 33.2 mm to (123.5, 82.0)
- moved J5 29.3 mm to (121.1, 92.7)
- moved U5 23.8 mm to (124.5, 86.3), turned to 90 degrees
- moved R7 21.2 mm to (105.2, 90.1), turned to 90 degrees
- moved C5 20.1 mm to (108.2, 82.1), turned to 180 degrees
- moved C8 20.1 mm to (111.7, 78.3), turned to 0 degrees
- moved C9 18.6 mm to (125.0, 89.9), turned to 180 degrees
- moved U3 14.2 mm to (111.5, 88.2), turned to -90 degrees
- moved D2 13.8 mm to (105.2, 86.6), turned to 90 degrees
- moved C7 13.2 mm to (112.6, 82.0), turned to 0 degrees
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Connections:
- C11 pad 2: GND -> GND1
- C12 pad 2: GND -> GND1
- C6 pad 2: GND -> GND1
- C9 pad 2: GND -> GND1
Routing:
- net /SDA: track 0.00 -> 31.2 mm, vias 0 -> 1
- net /UART_Tx: track 0.00 -> 29.0 mm
- net /UART_Rx: track 0.00 -> 27.8 mm
- net /SCL: track 0.00 -> 27.4 mm, vias 0 -> 1
- net /5V_ISO: track 0.00 -> 24.1 mm
- net /3V3_ISO: track 0.00 -> 17.1 mm, vias 0 -> 56
- net /LED_R: track 0.00 -> 14.8 mm
- net /LED_G: track 0.00 -> 12.0 mm
- net /BUZZER: track 0.00 -> 10.8 mm
- net /DAC_OUT: track 0.00 -> 7.28 mm
- net /SDA_ISO: track 0.00 -> 7.25 mm, vias 0 -> 3
- net /SCL_ISO: track 0.00 -> 7.23 mm, vias 0 -> 3
- net +5V: track 0.00 -> 7.10 mm
- net Net-(D1-A2): track 0.00 -> 4.76 mm
- net Net-(D1-A1): track 0.00 -> 4.76 mm
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- added copper zone on F.Cu, net +3.3V
- added copper zone on In1.Cu, net +3.3V
- added copper zone on F.Cu, net /3V3_ISO
- added copper zone on In1.Cu, net /3V3_ISO
- added copper zone on F.Cu, net GND
- added copper zone on In2.Cu, net GND
- added copper zone on F.Cu, net GND1
- added copper zone on In2.Cu, net GND1
- added copper zone on F.Cu, net Net-(U1-Vin)
Other:
- outline, holes or cut-outs redrawn
- copper layers 2 -> 4
- board text added: "DAC"

Commit message: Updated Layout, added UART + I2C headers
Parts:
- moved J3 35.7 mm to (130.7, 93.2), turned to 90 degrees
- moved J6 22.3 mm to (160.8, 80.2), turned to 0 degrees
- moved J4 12.1 mm to (149.5, 93.4), turned to 180 degrees
- moved J2 1.95 mm to (154.1, 77.6)
- moved C1 1.81 mm to (127.6, 60.3)
- moved C10 1.81 mm to (137.0, 60.2)
- moved C11 1.81 mm to (137.0, 71.0)
- moved C12 1.81 mm to (127.6, 71.0)
- moved R3 1.81 mm to (124.9, 58.9)
- moved R4 1.81 mm to (123.2, 58.9)
- moved R6 1.81 mm to (123.3, 73.4)
- moved U2 1.81 mm to (124.1, 65.7)
- moved U6 1.81 mm to (133.6, 65.7)
- moved R5 1.80 mm to (124.9, 73.4)
- moved D3 0.28 mm to (136.6, 52.0)
Connections:
- J3 pad 3: /ADC_AIN2 -> /ADC_AIN3
- J3 pad 4: /ADC_AIN3 -> /ADC_AIN2
Routing:
- net /SDA_ISO: track 7.25 -> 59.2 mm, vias 3 -> 5
- net /SCL_ISO: track 7.23 -> 58.5 mm, vias 3 -> 5
- net /UART_Tx_ISO: track 2.91 -> 40.0 mm
- net /UART_Rx_ISO: track 2.89 -> 36.0 mm
- net /ADC_AIN3: track 0.00 -> 9.00 mm
- net /ADC_AIN2: track 0.00 -> 8.60 mm
- net /ADC_AIN0: track 0.00 -> 7.88 mm
- net /ADC_AIN1: track 0.00 -> 7.55 mm
- net /SCL: track 27.4 -> 24.4 mm
- net /SDA: track 31.2 -> 29.6 mm
- net GND1: track 3.26 -> 4.76 mm, vias 46 -> 52
- net /UART_Rx: track 27.8 -> 26.4 mm
- net /UART_Tx: track 29.0 -> 27.7 mm
Other:
- outline, holes or cut-outs redrawn
- board text added: "3V3"
- board text added: "AIN0"
- board text added: "AIN1"
- board text added: "AIN2"
- board text added: "AIN3"
- board text added: "Designed By: Omar Mekkawy"
- board text added: "G"
- board text added: "RPi HW Automation HAT"
- board text added: "Rx"
- board text added: "SCL"
- board text added: "SDA"
- board text added: "Tx"

Commit message: Connected LED D3 to GPIO 16
Parts:
- moved D3 9.33 mm to (140.6, 60.4), turned to 90 degrees
- moved R11 4.61 mm to (140.6, 56.6), turned to -90 degrees
- moved R2 0.80 mm to (148.9, 55.2)
- moved R1 0.79 mm to (143.8, 55.2)
- moved D1 0.68 mm to (148.9, 60.4)
- moved C11 0.20 mm to (137.0, 71.2)
- moved C12 0.20 mm to (127.6, 71.2)
Connections:
- J1 pad 36: unconnected-(J1-GPIO16-Pad36) -> /LED_O
Routing:
- net /LED_O: track 0.00 -> 16.8 mm
- net Net-(D3-A): track 0.00 -> 2.04 mm
- net GND: track 2.00 -> 3.46 mm, vias 14 -> 12
- net GND1: vias 52 -> 47
- net /3V3_ISO: vias 56 -> 55
Other:
- outline, holes or cut-outs redrawn
